File: flight-controller.kicad_pcb (KiCad board)
At the start: 4 copper layers, 29 x 43 mm, 50 parts, among them J1 USB_C_Receptacle_USB2.0_16P, J2 Conn_Coaxial, J4 TC2030, SW1 SW_Push, U1 MIC5365-3.3YD5, U2 USBLC6-2SC6, U3 DLF162500LT-5028A1, U4 STM32WB55CEUx, U5 MPU-6050, X1 32kHz768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

Commit message: added test points
Parts:
- added TP1: TestPoint, TestPoint:TestPoint_Pad_D1.0mm, F.Cu at (88.2, 100.5)
- added TP2: TestPoint, TestPoint:TestPoint_Pad_D1.0mm, F.Cu at (93.8, 108.5)
- moved C13 0.21 mm to (101.0, 88.7)
Routing:
- net GND: track 35.1 -> 38.5 mm
- net /I2C1_SDA: track 20.3 -> 20.9 mm
