File: flight-controller.kicad_sch (KiCad schematic)
At the start: 50 parts, among them J1 USB_C_Receptacle_USB2.0_16P, J2 Conn_Coaxial, J4 TC2030, SW1 SW_Push, U1 MIC5365-3.3YD5, U2 USBLC6-2SC6, U3 DLF162500LT-5028A1, U4 STM32WB55CEUx, U5 MPU-6050, X1 32kHz768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

Commit message: almost no DRC errors
Parts:
- H1, H2, H3, H4: footprint MountingHole:MountingHole_2.2mm_M2 -> MountingHole:MountingHole_2.2mm_M2_Pad
Changed lines of the file:
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@@
 			)
 		)
-		(property "Footprint" "MountingHole:MountingHole_2.2mm_M2"
+		(property "Footprint" "MountingHole:MountingHole_2.2mm_M2_Pad"
 			(at 36.83 170.18 0)
 			(effects
@@
 		)
 		(instances
-			(project ""
+			(project "flight-controller"
 				(path "/a5f7a25c-082f-4bc5-b533-7e16fdbf1e58"
 					(reference "C21")
@@
 		)
 		(instances
-			(project ""
+			(project "flight-controller"
 				(path "/a5f7a25c-082f-4bc5-b533-7e16fdbf1e58"
 					(reference "#PWR025")
@@
 		)
 		(instances
-			(project ""
+			(project "flight-controller"
 				(path "/a5f7a25c-082f-4bc5-b533-7e16fdbf1e58"
 					(reference "R5")
@@
 		)
 		(instances
-			(project ""
+			(project "flight-controller"
 				(path "/a5f7a25c-082f-4bc5-b533-7e16fdbf1e58"
 					(reference "#PWR029")
@@
 		)
 		(instances
-			(project ""
+			(project "flight-controller"
 				(path "/a5f7a25c-082f-4bc5-b533-7e16fdbf1e58"
 					(reference "U5")
@@
 		)
 		(instances
-			(project ""
+			(project "flight-controller"
 				(path "/a5f7a25c-082f-4bc5-b533-7e16fdbf1e58"
 					(reference "#PWR026")
@@
 		)
 		(instances
-			(project ""
+			(project "flight-controller"
 				(path "/a5f7a25c-082f-4bc5-b533-7e16fdbf1e58"
 					(reference "#FLG02")
@@
 		)
 		(instances
-			(project ""
+			(project "flight-controller"
 				(path "/a5f7a25c-082f-4bc5-b533-7e16fdbf1e58"
 					(reference "C20")
@@
 			)
 		)
-		(property "Footprint" "MountingHole:MountingHole_2.2mm_M2"
+		(property "Footprint" "MountingHole:MountingHole_2.2mm_M2_Pad"
 			(at 17.78 170.18 0)
 			(effects
@@
 		)
 		(instances
-			(project ""
+			(project "flight-controller"
 				(path "/a5f7a25c-082f-4bc5-b533-7e16fdbf1e58"
 					(reference "H1")
@@
 			)
 		)
-		(property "Footprint" "MountingHole:MountingHole_2.2mm_M2"
+		(property "Footprint" "MountingHole:MountingHole_2.2mm_M2_Pad"
 			(at 27.94 170.18 0)
 			(effects
@@
 		)
 		(instances
-			(project ""
+			(project "flight-controller"
 				(path "/a5f7a25c-082f-4bc5-b533-7e16fdbf1e58"
 					(reference "#PWR028")
@@
 			)
 		)
-		(property "Footprint" "MountingHole:MountingHole_2.2mm_M2"
+		(property "Footprint" "MountingHole:MountingHole_2.2mm_M2_Pad"
 			(at 45.72 170.18 0)
 			(effects
@@
 		)
 		(instances
-			(project ""
+			(project "flight-controller"
 				(path "/a5f7a25c-082f-4bc5-b533-7e16fdbf1e58"
 					(reference "#PWR030")
@@
 		)
 		(instances
-			(project ""
+			(project "flight-controller"
 				(path "/a5f7a25c-082f-4bc5-b533-7e16fdbf1e58"
 					(reference "#PWR027")
@@
 		)
 		(instances
-			(project ""
+			(project "flight-controller"
 				(path "/a5f7a25c-082f-4bc5-b533-7e16fdbf1e58"
 					(reference "C23")
@@
 		)
 		(instances
-			(project ""
+			(project "flight-controller"
 				(path "/a5f7a25c-082f-4bc5-b533-7e16fdbf1e58"
 					(reference "X2")
@@
 		)
 		(instances
-			(project ""
+			(project "flight-controller"
 				(path "/a5f7a25c-082f-4bc5-b533-7e16fdbf1e58"
 					(reference "#PWR019")
@@
 		)
 		(instances
-			(project ""
+			(project "flight-controller"
 				(path "/a5f7a25c-082f-4bc5-b533-7e16fdbf1e58"
 					(reference "#FLG01")
@@
 		)
 		(instances
-			(project ""
+			(project "flight-controller"
 				(path "/a5f7a25c-082f-4bc5-b533-7e16fdbf1e58"
 					(reference "J4")
@@
 		)
 		(instances
-			(project ""
+			(project "flight-controller"
 				(path "/a5f7a25c-082f-4bc5-b533-7e16fdbf1e58"
 					(reference "C22")
@@
 		)
 		(instances
-			(project ""
+			(project "flight-controller"
 				(path "/a5f7a25c-082f-4bc5-b533-7e16fdbf1e58"
 					(reference "FID1")

Commit message: added test points
Parts:
- added TP1, TP2: TestPoint, TestPoint:TestPoint_Pad_D1.0mm, symbol Connector:TestPoint
Connections:
- net I2C1_SCL: now also TP1.1
- net I2C1_SDA: now also TP2.1
Changed lines of the file:
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@@
 	)
 	(junction
+		(at 100.33 123.19)
+		(diameter 0)
+		(color 0 0 0 0)
+	)
+	(junction
 		(at 101.6 162.56)
 		(diameter 0)
@@
 	)
 	(junction
+		(at 86.36 120.65)
+		(diameter 0)
+		(color 0 0 0 0)
+	)
+	(junction
 		(at 109.22 30.48)
 		(diameter 0)
@@
 	(wire
 		(pts
-			(xy 105.41 123.19) (xy 88.9 123.19)
+			(xy 105.41 123.19) (xy 100.33 123.19)
 		)
 		(stroke
@@
 	(wire
 		(pts
+			(xy 100.33 116.84) (xy 100.33 123.19)
+		)
+		(stroke
+			(width 0)
+			(type default)
+		)
+	)
+	(wire
+		(pts
 			(xy 176.53 100.33) (xy 175.26 100.33)
 		)
@@
 	(wire
 		(pts
+			(xy 100.33 123.19) (xy 88.9 123.19)
+		)
+		(stroke
+			(width 0)
+			(type default)
+		)
+	)
+	(wire
+		(pts
 			(xy 27.94 175.26) (xy 36.83 175.26)
 		)
@@
 	(wire
 		(pts
+			(xy 86.36 116.84) (xy 86.36 120.65)
+		)
+		(stroke
+			(width 0)
+			(type default)
+		)
+	)
+	(wire
+		(pts
 			(xy 176.53 114.3) (xy 176.53 116.84)
 		)
@@
 	)
 	(symbol
+		(lib_id "Connector:TestPoint")
+		(at 100.33 116.84 0)
+		(unit 1)
+		(exclude_from_sim no)
+		(in_bom yes)
+		(on_board yes)
+		(dnp no)
+		(fields_autoplaced yes)
+		(property "Reference" "TP2"
+			(at 102.87 112.2679 0)
+			(effects
+				(font
+					(size 1.27 1.27)
+				)
+				(justify left)
+			)
+		)
+		(property "Value" "TestPoint"
+			(at 102.87 114.8079 0)
+			(effects
+				(font
+					(size 1.27 1.27)
+				)
+				(justify left)
+			)
+		)
+		(property "Footprint" "TestPoint:TestPoint_Pad_D1.0mm"
+			(at 105.41 116.84 0)
+			(effects
+				(font
+					(size 1.27 1.27)
+				)
+				(hide yes)
+			)
+		)
+		(property "Datasheet" "~"
+			(at 105.41 116.84 0)
+			(effects
+				(font
+					(size 1.27 1.27)
+				)
+				(hide yes)
+			)
+		)
+		(property "Description" "test point"
+			(at 100.33 116.84 0)
+			(effects
+				(font
+					(size 1.27 1.27)
+				)
+				(hide yes)
+			)
+		)
+		(pin "1"
+		)
+		(instances
+			(project ""
+				(path "/a5f7a25c-082f-4bc5-b533-7e16fdbf1e58"
+					(reference "TP2")
+					(unit 1)
+				)
+			)
+		)
+	)
+	(symbol
 		(lib_id "power:GND")
 		(at 73.66 114.3 0)
@@
 					(unit 1)
 				)
+			)
+		)
+	)
+	(symbol
+		(lib_id "Connector:TestPoint")
+		(at 86.36 116.84 0)
+		(unit 1)
+		(exclude_from_sim no)
+		(in_bom yes)
+		(on_board yes)
+		(dnp no)
+		(fields_autoplaced yes)
+		(property "Reference" "TP1"
+			(at 88.9 112.2679 0)
+			(effects
+				(font
+					(size 1.27 1.27)
+				)
+				(justify left)
+			)
+		)
+		(property "Value" "TestPoint"
+			(at 88.9 114.8079 0)
+			(effects
+				(font
+					(size 1.27 1.27)
+				)
+				(justify left)
+			)
+		)
+		(property "Footprint" "TestPoint:TestPoint_Pad_D1.0mm"
+			(at 91.44 116.84 0)
+			(effects
+				(font
+					(size 1.27 1.27)
+				)
+				(hide yes)
+			)
+		)
+		(property "Datasheet" "~"
+			(at 91.44 116.84 0)
+			(effects
+				(font
+					(size 1.27 1.27)
+				)
+				(hide yes)
+			)
+		)
+		(property "Description" "test point"
+			(at 86.36 116.84 0)
+			(effects
+				(font
+					(size 1.27 1.27)
+				)
+				(hide yes)
+			)
+		)
+		(pin "1"
+		)
+		(instances
+			(project ""
+				(path "/a5f7a25c-082f-4bc5-b533-7e16fdbf1e58"
+					(reference "TP1")
+					(unit 1)
+				)
